File: schematics/Orion68/_autosave-ide.kicad_sch (KiCad schematic)
At the start: 2 parts, among them J5 Euro96pin, U31 GAL20V8

Commit message: Changed dtack system
Connections:
- net /CS_MULTIIO: now also U31.2 (I); no longer U31.4 (I)
- net /DTACK_SMIO: now also U31.4 (I); no longer U31.2 (I)
Changed lines of the file:
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@@
 	)
 	(label "{slash}CS_MULTIIO"
-		(at 41.91 38.1 180)
+		(at 41.91 33.02 180)
 		(effects
 			(font
@@
 	)
 	(label "{slash}DTACK_SMIO"
-		(at 41.91 33.02 180)
+		(at 41.91 38.1 180)
 		(effects
 			(font
