File: schematics/Orion68/orion68_serial.kicad_sch (KiCad schematic)
At the start: 65 parts, among them J11 IDE-40W, J12 PWR, J700 Euro96pin, J701 RS232_1, J702 RS232_1, J703 RS232_1, U17 74LS139, U18_C? 100nf, U19 74LS139, U20 74HC138, U701 UART1, U702 UART2, U703 UART3, Y1 14.745600

Commit message: Power control implemented
Connections:
- net IORDY: now reaches J11.27 (Pin_27), R54.1
- net INTRQ: now reaches J11.31 (Pin_31), R53.1
Changed lines of the file:
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@@
 	(wire
 		(pts
-			(xy 119.38 236.22) (xy 149.86 236.22)
+			(xy 111.76 236.22) (xy 149.86 236.22)
 		)
 		(stroke
@@
 	(wire
 		(pts
-			(xy 119.38 223.52) (xy 124.46 223.52)
+			(xy 111.76 223.52) (xy 124.46 223.52)
 		)
 		(stroke
@@
 	(wire
 		(pts
-			(xy 119.38 223.52) (xy 119.38 236.22)
+			(xy 111.76 223.52) (xy 111.76 236.22)
 		)
 		(stroke
@@
 		)
 	)
+	(label "IORDY"
+		(at 104.14 208.28 0)
+		(effects
+			(font
+				(size 1.27 1.27)
+			)
+			(justify left bottom)
+		)
+	)
 	(label "RXC"
 		(at 187.96 92.71 0)
@@
 		)
 	)
+	(label "INTRQ"
+		(at 104.14 213.36 0)
+		(effects
+			(font
+				(size 1.27 1.27)
+			)
+			(justify left bottom)
+		)
+	)
