File: schematics/Orion68/orion68vid.kicad_sch (KiCad schematic)
At the start: 29 parts, among them J300 Euro96pin, Q4 2N7000, U301 74HC245, U302 74HC245, U303 24LC256, U304 GAL16V8, U305 74LS541

Commit message: Implemented new picoVGA V2
Parts:
- removed Q4: 2N7000, Package_TO_SOT_THT:TO-92_Inline, symbol Transistor_FET:2N7000
- removed R300, R301, R302, R303, R304, R305, R306, R307, R308, R309, R310, R311, R312, R318: 1k, Resistor_THT:R_Axial_DIN0204_L3.6mm_D1.6mm_P5.08mm_Horizontal, symbol Device:R
- removed R316: 10K, Resistor_THT:R_Axial_DIN0204_L3.6mm_D1.6mm_P5.08mm_Horizontal, symbol Device:R
- removed R317: 10k, Resistor_THT:R_Axial_DIN0204_L3.6mm_D1.6mm_P5.08mm_Horizontal, symbol Device:R
- removed U301, U302: 74HC245, Package_DIP:DIP-20_W7.62mm, symbol 74xx:74HC245
- removed U303: 24LC256, Package_DIP:DIP-8_W7.62mm, symbol Memory_EEPROM:24LC256
- removed U305: 74LS541, symbol 74xx:74LS541
- added C16: 100nF, symbol Device:C
- added C17: 10uF, symbol Device:C_Polarized
- added J21: DE15_Socket_HighDensity, symbol Connector:DE15_Socket_HighDensity
- added U301, U302: SN74LVC245APW, Package_SO:TSSOP-20_4.4x6.5mm_P0.65mm, symbol Logic_LevelTranslator:SN74LVC245APW
- added U32: ~, Package_TO_SOT_SMD:TO-252-3_TabPin2, symbol Regulator_Linear:LM1117DT-1.8
- U300: value ~ -> Multio
Connections:
- net A08 is gone; now on net A11: U304.4 (I4)
- net A09 is gone; now on net A10: U304.3 (I3)
- net BA15 is gone; now on net A8: U304.1 (I1/CLK)
- net B/AS is gone; now on net A15: U304.8 (I8)
- net SDA is gone; now on net /DTACK_PVGA: U300.19 (GP14)
- net +5V: now also C16.1, U32.3 (VI); no longer U300.39 (VSYS)
- net A1: now also U302.18 (B1)
- net A10: no longer U304.2 (I2)
- net A11: no longer U304.6 (I6)
- net A12: now also U304.5 (I5); no longer U304.14 (IO6)
- net A13: now also U304.6 (I6); no longer U304.13 (IO7)
- net A14: now also U304.7 (I7); no longer U304.11 (I10/~{OE})
- net A2: now also U302.17 (B2)
- net A3: now also U302.16 (B3)
- net A4: now also U302.15 (B4)
- net A5: now also U302.14 (B5)
- net A6: now also U302.13 (B6)
- net A9: now also U304.2 (I2)
- net BLUE: now also J21.3
- net D0: now also U301.18 (B1); no longer U300.1 (GP0)
- net D1: now also U301.17 (B2); no longer U300.2 (GP1)
- net D2: now also U301.16 (B3); no longer U300.4 (GP2)
- net D3: now also U301.15 (B4); no longer U300.5 (GP3)
- net D4: now also U301.14 (B5); no longer U300.6 (GP4)
- net D5: now also U301.13 (B6); no longer U300.7 (GP5)
- net D6: now also U301.12 (B7); no longer U300.9 (GP6)
- net D7: now also U301.11 (B8); no longer U300.10 (GP7)
- net GND: now also C16.2, C17.2, J21.10, J21.5, J21.6, J21.7, J21.8, U301.10 (GND), U302.1 (DIR), U302.10 (GND), U302.19 (~{OE}), U32.1 (GND)
- net GREEN: now also J21.2
- net HSYNC: now also J21.13
- net Red: now also J21.1
- net VSYNC: now also J21.14
- net /AS: now also U304.12 (IO8)
- net /IO_CS1: now also U304.11 (I10/~{OE}); no longer U304.5 (I5)
- net /iord: now also U304.14 (IO6); no longer U304.16 (IO4)
- net /iowr: now also U304.13 (IO7); no longer U304.7 (I7)
- net /memwr: now also U301.1 (DIR), U302.12 (B7)
- net VERMELHO: now reaches U304.19 (IO1)
- net VERMELHO: now also J300.58, U301.19 (~{OE}), U302.11 (B8)
- net PRETO: now reaches J300.57
- net /DTACK_PVGA: now reaches J300.59
- net MARRON: now reaches J300.60
- net AMARELO: now reaches J300.61
- net VERDE: now reaches J300.62
- net LILAS: now reaches J300.63
- net A1_C: now reaches U300.11 (GP8)
- net A1_C: now also U302.2 (A1)
- net A2_C: now reaches U300.12 (GP9)
- net A2_C: now also U302.3 (A2)
- net A3_C: now reaches U300.14 (GP10)
- net A3_C: now also U302.4 (A3)
- net A4_C: now reaches U300.15 (GP11)
- net A4_C: now also U302.5 (A4)
- net A5_C: now reaches U300.16 (GP12)
- net A5_C: now also U302.6 (A5)
- net 3V3: now reaches U300.39 (VSYS)
- net 3V3: now also C17.1, U301.20 (VCC), U302.20 (VCC), U32.2 (VO)
- net +3,3V: no longer names the net of U300.36 (3V3(OUT))
- net SCL renamed /WR_C
- net /WR_C: now also U302.8 (A7)
- net ST0 renamed /CS_PVGA_C
- net /CS_PVGA_C: now also U302.9 (A8)
- net ST1: no longer names the net of U300.29 (GP22)
- net ST2: no longer names the net of U300.31 (GP26)
- net ST3: no longer names the net of U300.32 (GP27)
- net ST4: no longer names the net of U300.34 (GP28)
- net /CS renamed A6_C
- net A6_C: now also U302.7 (A6)
- net /ST_CS: no longer names the net of U304.18 (IO2)
- new net: U300.1 (GP0), U301.2 (A1)
- new net: U300.10 (GP7), U301.9 (A8)
- new net: U300.2 (GP1), U301.3 (A2)
- new net: U300.4 (GP2), U301.4 (A3)
- new net: U300.5 (GP3), U301.5 (A4)
- new net: U300.6 (GP4), U301.6 (A5)
- new net: U300.7 (GP5), U301.7 (A6)
- new net: U300.9 (GP6), U301.8 (A7)
- no-connect marks 0 -> 9
Other:
- note added: "LILAS"
- note added: "dir = 1 A -> B dir = 0 B -> A"
- note removed: "74HC245 B -> A pino 1 = GND A -> B pino 1 = VCC"
- note removed: "NÃO IMPLEMENTADO NOT IMPLEMENTED"
- moved on the sheet: R313, R314, R315, U304

Commit message: W5100 running with direct socket
Connections:
- net A16: now also U304.13 (IO7)
- net A17: now also U304.14 (IO6)
- net A18: now also U304.15 (IO5)
- net A19: now also U304.16 (IO4)
- net /AS: now also U304.17 (I03); no longer U304.12 (IO8)
- net /iord: no longer U304.14 (IO6)
- net /iowr: no longer U304.13 (IO7)
- net /CS_W5100: now reaches U304.18 (IO2)
Changed lines of the file:
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@@
+	(wire
+		(pts
+			(xy 212.09 97.79) (xy 218.44 97.79)
+		)
+		(stroke
+			(width 0)
+			(type default)
+		)
+	)
 	(wire
 		(pts
@@
 		)
 	)
+	(label "{slash}CS_W5100"
+		(at 212.09 97.79 180)
+		(effects
+			(font
+				(size 1.27 1.27)
+			)
+			(justify right bottom)
+		)
+	)
 	(label "{slash}AS"
-		(at 218.44 113.03 180)
+		(at 218.44 100.33 180)
 		(effects
 			(font
@@
 		)
 	)
+	(label "A18"
+		(at 218.44 105.41 180)
+		(effects
+			(font
+				(size 1.27 1.27)
+			)
+			(justify right bottom)
+		)
+	)
 	(label "D2"
 		(at 19.05 74.93 0)
@@
 		)
 	)
+	(label "A19"
+		(at 218.44 102.87 180)
+		(effects
+			(font
+				(size 1.27 1.27)
+			)
+			(justify right bottom)
+		)
+	)
 	(label "A6"
 		(at 81.28 154.94 180)
@@
 		)
 	)
+	(label "A17"
+		(at 218.44 107.95 180)
+		(effects
+			(font
+				(size 1.27 1.27)
+			)
+			(justify right bottom)
+		)
+	)
 	(label "{slash}iord"
 		(at 40.64 85.09 0)
@@
 		)
 	)
-	(label "{slash}iord"
-		(at 218.44 107.95 180)
-		(effects
-			(font
-				(size 1.27 1.27)
-			)
-			(justify right bottom)
-		)
-	)
 	(label "A13"
 		(at 250.19 107.95 0)
@@
 		)
 	)
-	(label "{slash}iowr"
-		(at 218.44 110.49 180)
-		(effects
-			(font
-				(size 1.27 1.27)
-			)
-			(justify right bottom)
-		)
-	)
 	(label "D3"
 		(at 71.12 92.71 180)
@@
 		(effects
 			(font
+				(size 1.27 1.27)
+			)
+			(justify right bottom)
+		)
+	)
+	(label "A16"
+		(at 218.44 110.49 180)
+		(effects
+			(font
